File: de10-lite-ram-rom.sch (KiCad schematic (older format))
At the start: 8 parts, among them J6 DE10-Lite GPIO, U1 AS6C4008A-55ZIN, U2 SST39LF040

Commit message: Final version
Parts:
- removed J6: DE10-Lite GPIO, Connector_PinSocket_2.54mm:PinSocket_2x20_P2.54mm_Vertical, symbol Connector_Generic:Conn_02x20_Odd_Even
- added J1: DE10-Lite_GPIO_Header, Connector_PinSocket_2.54mm:PinSocket_2x20_P2.54mm_Horizontal, symbol Connector_Generic:DE10-Lite_GPIO_Header
- U1: Description (none) -> SRAM 4M, 2.7-5.5V, 55ns 512K x 8 Asynch SRAM; MFR (none) -> Alliance Memory; MPN (none) -> AS6C4008A-55ZIN; SPN (none) -> 913-AS6C4008A-55ZIN; SPR (none) -> Mouser; SPURL (none) -> https://www.mouser.com/ProductDetail/Alliance-Memory/AS6C40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
- U2: Description NOR Flash 4.5 to 5.5 1Mbit Multi-Purpose Flash -> NOR Flash 3.0V to 3.6V 4Mbit Multi-Purpose Flash; SPURL https://www.mouser.com/datasheet/2/268/01360A-709051.pdf -> https://www.mouser.com/ProductDetail/Microchip-Technology/S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
Other:
- note added: "AA10"
- note added: "AA14"
- note added: "AA15"
- note added: "AA5"
- note added: "AA6"
- note added: "AA7"
- note added: "AA8"
- note added: "AA9"
- note added: "AB10"
- note added: "AB11"
- note added: "AB12"
- note added: "AB13"
- note added: "AB3"
- note added: "V5"
- note added: "V7"
- note added: "V8"
- note added: "W11"
- note added: "W12"
- note added: "W13"
- note added: "W5"
- note added: "W6"
- note added: "W7"
- note added: "W8"
- note added: "W9"
- note added: "Y11"
- note added: "Y3"
- note added: "Y4"
- note added: "Y5"
- note added: "Y6"
- note added: "Y7"
- note added: "Y8"
Changed lines of the file:
@@
 	3050 4300 2450 4300
 Wire Wire Line
-	3450 4500 2450 4500
+	3450 4500 3250 4500
 Wire Wire Line
 	1950 5400 1050 5400
-Wire Wire Line
-	3450 5400 3300 5400
 $Comp
 L power:GND #PWR027
@@
 F 2 "Package_LCC:PLCC-32_11.4x14.0mm_P1.27mm-Socket" H 9500 2400 50  0001 C CNN
 F 3 "https://www.mouser.com/datasheet/2/268/01360A-709051.pdf" H 9500 2400 50  0001 C CNN
-F 4 "NOR Flash 4.5 to 5.5 1Mbit Multi-Purpose Flash" H 9500 2100 50  0001 C CNN "Description"
+F 4 "NOR Flash 3.0V to 3.6V 4Mbit Multi-Purpose Flash" H 9500 2100 50  0001 C CNN "Description"
 F 5 "Microchip" H 9500 2100 50  0001 C CNN "MFR"
 F 6 "SST39LF040-55-4C-NHE-T" H 9500 2100 50  0001 C CNN "MPN"
 F 7 "579-SST39LF040554CN" H 9500 2100 50  0001 C CNN "SPN"
 F 8 "Mouser" H 9500 2100 50  0001 C CNN "SPR"
-F 9 "https://www.mouser.com/datasheet/2/268/01360A-709051.pdf" H 9500 2100 50  0001 C CNN "SPURL"
+F 9 "https://www.mouser.com/ProductDetail/Microchip-Technology/SST39LF040-55-4C-NHE-T?qs=%2Fha2pyFaduhPPB5QetWHjyzBss7yQNcI4yvsI8zP%2F3nbLSqNwKNiLbVcDmJEYEkq" H 9500 2100 50  0001 C CNN "SPURL"
 	1    9500 2100
 	1    0    0    -1
@@
 	1    0    0    -1
 $EndComp
-$Comp
-L power:PWR_FLAG #FLG03
-U 1 1 5D96378E
-P 3300 5400
-F 0 "#FLG03" H 3300 5475 50  0001 C CNN
-F 1 "PWR_FLAG" H 3300 5573 50  0000 C CNN
-F 2 "" H 3300 5400 50  0001 C CNN
-F 3 "~" H 3300 5400 50  0001 C CNN
-	1    3300 5400
-	1    0    0    -1
-$EndComp
-$Comp
-L power:PWR_FLAG #FLG02
-U 1 1 5D964468
-P 1050 5400
-F 0 "#FLG02" H 1050 5475 50  0001 C CNN
-F 1 "PWR_FLAG" H 1050 5573 50  0000 C CNN
-F 2 "" H 1050 5400 50  0001 C CNN
-F 3 "~" H 1050 5400 50  0001 C CNN
-	1    1050 5400
-	0    -1   -1   0
-$EndComp
 Wire Wire Line
 	6650 2100 5800 2100
@@
 	1950 4500 1000 4500
 $Comp
-L power:PWR_FLAG #FLG01
-U 1 1 5D95CB67
-P 1000 4500
-F 0 "#FLG01" H 1000 4575 50  0001 C CNN
-F 1 "PWR_FLAG" H 1000 4673 50  0000 C CNN
-F 2 "" H 1000 4500 50  0001 C CNN
-F 3 "~" H 1000 4500 50  0001 C CNN
-	1    1000 4500
-	0    -1   -1   0
-$EndComp
-$Comp
 L power:VCC #PWR030
 U 1 1 5D95CB6D
@@
 Text Label 1350 4500 0    50   ~ 0
 5V
-$Comp
-L Connector_Generic:Conn_02x20_Odd_Even J6
-U 1 1 5D754F95
-P 2150 4900
-F 0 "J6" H 2200 6017 50  0000 C CNN
-F 1 "DE10-Lite GPIO" H 2200 5926 50  0000 C CNN
-F 2 "Connector_PinSocket_2.54mm:PinSocket_2x20_P2.54mm_Vertical" H 2150 4900 50  0001 C CNN
-F 3 "~" H 2150 4900 50  0001 C CNN
-	1    2150 4900
-	1    0    0    -1
-$EndComp
 Wire Wire Line
 	5800 2200 6400 2200
@@
 Wire Wire Line
 	3050 4700 2450 4700
-Connection ~ 3300 5400
 Wire Wire Line
 	3050 5000 2450 5000
 Wire Wire Line
 	2450 4200 3050 4200
-Wire Wire Line
-	3300 5400 2450 5400
 $Comp
 L Device:C_Small C4
@@
 	1    0    0    -1
 $EndComp
-Connection ~ 1000 4500
 NoConn ~ 1950 5900
 Wire Wire Line
@@
 F 1 "AS6C4008A-55ZIN" H 5750 3100 50  0000 C CNN
 F 2 "Package_SO:TSOP-II-32_21.0x10.2mm_P1.27mm" H 5300 2100 50  0001 C CNN
-F 3 "" H 5300 2100 50  0001 C CNN
+F 3 "https://www.mouser.com/datasheet/2/12/AS6C4008A-1288404.pdf" H 5300 2100 50  0001 C CNN
+F 4 "SRAM 4M, 2.7-5.5V, 55ns 512K x 8 Asynch SRAM" H 5300 2000 50  0001 C CNN "Description"
+F 5 "Alliance Memory" H 5300 2000 50  0001 C CNN "MFR"
+F 6 "AS6C4008A-55ZIN" H 5300 2000 50  0001 C CNN "MPN"
+F 7 "913-AS6C4008A-55ZIN" H 5300 2000 50  0001 C CNN "SPN"
+F 8 "Mouser" H 5300 2000 50  0001 C CNN "SPR"
+F 9 "https://www.mouser.com/ProductDetail/Alliance-Memory/AS6C4008A-55ZIN?qs=sGAEpiMZZMt9mBA6nIyysK%252B2%2Fppis4NuiMdKv%2FEcOn8%3D" H 5300 2000 50  0001 C CNN "SPURL"
 	1    5300 2000
 	1    0    0    -1
@@
 	1950 4900 1350 4900
 NoConn ~ 2450 4000
+Text Notes 2550 4100 0    50   ~ 0
+W9
+Text Notes 2550 4200 0    50   ~ 0
+W8
+Text Notes 2550 4300 0    50   ~ 0
+W7
+Text Notes 2550 4400 0    50   ~ 0
+V5
+Text Notes 2550 4600 0    50   ~ 0
+AA15
+Text Notes 2550 4700 0    50   ~ 0
+W13
+Text Notes 2550 4800 0    50   ~ 0
+AB13
+Text Notes 2550 4900 0    50   ~ 0
+Y11
+Text Notes 2550 5000 0    50   ~ 0
+W11
+Text Notes 2550 5100 0    50   ~ 0
+AA10
+Text Notes 2550 5200 0    50   ~ 0
+Y8
+Text Notes 2550 5300 0    50   ~ 0
+Y7
+Text Notes 2550 5500 0    50   ~ 0
+Y6
+Text Notes 2550 5600 0    50   ~ 0
+Y5
+Text Notes 2550 5700 0    50   ~ 0
+Y4
+Text Notes 2550 5800 0    50   ~ 0
+Y3
+Text Notes 1600 5800 0    50   ~ 0
+AB3
+Text Notes 1600 5700 0    50   ~ 0
+AA5
+Text Notes 1600 5600 0    50   ~ 0
+AA6
+Text Notes 1600 5500 0    50   ~ 0
+AA7
+Text Notes 1600 5300 0    50   ~ 0
+AA8
+Text Notes 1600 5200 0    50   ~ 0
+AA9
+Text Notes 1600 5100 0    50   ~ 0
+AB10
+Text Notes 1600 5000 0    50   ~ 0
+AB11
+Text Notes 1600 4900 0    50   ~ 0
+AB12
+Text Notes 1600 4800 0    50   ~ 0
+W12
+Text Notes 1600 4700 0    50   ~ 0
+AA14
+Text Notes 1600 4600 0    50   ~ 0
+W5
+Text Notes 1600 4400 0    50   ~ 0
+W6
+Text Notes 1600 4300 0    50   ~ 0
+V7
+Text Notes 1600 4200 0    50   ~ 0
+V8
+$Comp
+L Connector_Generic:DE10-Lite_GPIO_Header J1
+U 1 1 5EA932AA
+P 2150 4900
+F 0 "J1" H 2200 6017 50  0000 C CNN
+F 1 "DE10-Lite_GPIO_Header" H 2200 5926 50  0000 C CNN
+F 2 "Connector_PinSocket_2.54mm:PinSocket_2x20_P2.54mm_Horizontal" H 2150 4900 50  0001 C CNN
+F 3 "~" H 2150 4900 50  0001 C CNN
+	1    2150 4900
+	1    0    0    -1
+$EndComp
+Wire Wire Line
+	2450 5400 3450 5400
+$Comp
+L power:PWR_FLAG #FLG0101
+U 1 1 5EAD2017
+P 3250 4500
+F 0 "#FLG0101" H 3250 4575 50  0001 C CNN
+F 1 "PWR_FLAG" H 3250 4673 50  0000 C CNN
+F 2 "" H 3250 4500 50  0001 C CNN
+F 3 "~" H 3250 4500 50  0001 C CNN
+	1    3250 4500
+	1    0    0    -1
+$EndComp
+Connection ~ 3250 4500
+Wire Wire Line
+	3250 4500 2450 4500
 $EndSCHEMATC

Commit message: removed pullups
Parts:
- removed R2, R7: 10K, Resistor_SMD:R_0603_1608Metric_Pad1.05x0.95mm_HandSolder, symbol Device:R_Small
- J1: symbol Connector_Generic:DE10-Lite_GPIO_Header -> de10-lite-ram-rom-rescue:DE10-Lite_GPIO_Header-Connector_Generic
Connections:
- wire segments 105 -> 104
Changed lines of the file:
@@
 $EndComp
 Wire Wire Line
-	6650 2100 5800 2100
-$Comp
-L Device:R_Small R7
-U 1 1 5D990AA4
-P 7800 3000
-F 0 "R7" H 7859 3046 50  0000 L CNN
-F 1 "10K" V 7800 2950 32  0000 L CNN
-F 2 "Resistor_SMD:R_0603_1608Metric_Pad1.05x0.95mm_HandSolder" H 7800 3000 50  0001 C CNN
-F 3 "~" H 7800 3000 50  0001 C CNN
-	1    7800 3000
-	1    0    0    -1
-$EndComp
-Wire Wire Line
-	7800 3100 8900 3100
-$Comp
-L Device:R_Small R2
-U 1 1 5D99EDEB
-P 6650 2000
-F 0 "R2" H 6709 2046 50  0000 L CNN
-F 1 "10K" H 6709 1955 50  0000 L CNN
-F 2 "Resistor_SMD:R_0603_1608Metric_Pad1.05x0.95mm_HandSolder" H 6650 2000 50  0001 C CNN
-F 3 "~" H 6650 2000 50  0001 C CNN
-	1    6650 2000
-	-1   0    0    -1
-$EndComp
+	6400 2100 5800 2100
+Wire Wire Line
+	8300 3100 8900 3100
 $Comp
 L power:VCC #PWR03
@@
 Text Label 3050 5400 2    50   ~ 0
 GND
-$Comp
-L power:VCC #PWR014
-U 1 1 5DA50D5B
-P 7800 2900
-F 0 "#PWR014" H 7800 2750 50  0001 C CNN
-F 1 "VCC" H 7817 3073 50  0000 C CNN
-F 2 "" H 7800 2900 50  0001 C CNN
-F 3 "" H 7800 2900 50  0001 C CNN
-	1    7800 2900
-	1    0    0    -1
-$EndComp
 Text Notes 9350 2250 0    50   ~ 0
 512K Flash
@@
 Wire Wire Line
 	5800 1800 6400 1800
-$Comp
-L power:VCC #PWR06
-U 1 1 5DBFE09F
-P 6650 1850
-F 0 "#PWR06" H 6650 1700 50  0001 C CNN
-F 1 "VCC" H 6667 2023 50  0000 C CNN
-F 2 "" H 6650 1850 50  0001 C CNN
-F 3 "" H 6650 1850 50  0001 C CNN
-	1    6650 1850
-	1    0    0    -1
-$EndComp
-Wire Wire Line
-	6650 1850 6650 1900
 Wire Wire Line
 	1950 4500 1000 4500
@@
 V8
 $Comp
-L Connector_Generic:DE10-Lite_GPIO_Header J1
+L de10-lite-ram-rom-rescue:DE10-Lite_GPIO_Header-Connector_Generic J1
 U 1 1 5EA932AA
 P 2150 4900
